Commit message: ball rendering!

File: urdf/dual_panda_example.urdf (robot description, URDF)
Before this commit: robot panda, 26 links, 25 joints
Links:
- link panda_2_paddle: geometry collision cylinder length=0.02 radius=0.25; visual cylinder length=0.02 radius=0.15
Joints:
- joint panda_2_paddle_joint: origin xyz=0 0 0.1 rpy=0 0 0 -> xyz=0 0 0.25 rpy=0 0 0

Commit message: recording condition, joint states, and ball functionality, nf for negating x-y component

File: urdf/dual_panda_example.urdf (robot description, URDF)
Before this commit: robot panda, 26 links, 25 joints
Links:
- link panda_2_paddle: geometry collision cylinder length=0.02 radius=0.25; visual cylinder length=0.02 radius=0.25
